File: Mae_Keyboard_Dev_Kit/Atreus62.kicad_sch (KiCad schematic)
At the start: 139 parts, among them J1 gc9a01_DISPLAY, J2 Conn_01x11_Pin, SW1 SWITCH_PUSH, SW10 SWITCH_PUSH, SW11 SWITCH_PUSH, SW12 SWITCH_PUSH, SW13 SWITCH_PUSH, SW14 SWITCH_PUSH, SW15 SWITCH_PUSH, SW16 SWITCH_PUSH, SW17 SWITCH_PUSH, SW18 SWITCH_PUSH, SW19 SWITCH_PUSH, SW2 SWITCH_PUSH, SW20 SWITCH_PUSH, SW21 SWITCH_PUSH, SW22 SWITCH_PUSH, SW23 SWITCH_PUSH, SW24 SWITCH_PUSH, SW25 SWITCH_PUSH, SW26 SWITCH_PUSH, SW27 SWITCH_PUSH, SW28 SWITCH_PUSH, SW29 SWITCH_PUSH, SW3 SWITCH_PUSH, SW30 SWITCH_PUSH, SW31 SWITCH_PUSH, SW32 SWITCH_PUSH, SW33 SWITCH_PUSH, SW34 SWITCH_PUSH, SW36 SWITCH_PUSH, SW37 SWITCH_PUSH, SW38 SWITCH_PUSH, SW39 SWITCH_PUSH, SW4 SWITCH_PUSH, SW40 SWITCH_PUSH, SW41 SWITCH_PUSH, SW42 SWITCH_PUSH, SW43 SWITCH_PUSH, SW44 SWITCH_PUSH, SW45 SWITCH_PUSH, SW46 SWITCH_PUSH, SW47 SWITCH_PUSH, SW48 SWITCH_PUSH, SW49 SWITCH_PUSH, SW5 SWITCH_PUSH, SW50 SWITCH_PUSH, SW51 SWITCH_PUSH, SW52 SWITCH_PUSH, SW53 SWITCH_PUSH, SW54 SWITCH_PUSH, SW55 SWITCH_PUSH, SW56 SWITCH_PUSH, SW57 SWITCH_PUSH, SW58 SWITCH_PUSH, SW59 SWITCH_PUSH, SW6 SWITCH_PUSH, SW60 SWITCH_PUSH, SW61 SWITCH_PUSH, SW62 SWITCH_PUSH, SW63 SWITCH_PUSH, SW64 SWITCH_PUSH, SW65 SWITCH_PUSH, SW7 SWITCH_PUSH, SW8 SWITCH_PUSH, SW9 SWITCH_PUSH, U3 ESP32-S3-DevKitC

Commit message: update
Parts:
- added TP1, TP2, TP3: TestPoint, TestPoint:TestPoint_Pad_4.0x4.0mm, symbol Connector:TestPoint
Connections:
- net +5V: now also TP2.1
- net CS: now also U3.41 (GPIO1/ADC1_CH0)
- net DC: now also U3.40 (GPIO2/ADC1_CH1)
- net GND: now also J2.2 (Pin_2), TP1.1
- net RST: now also U3.42 (GPIO44/U0RXD)
- net SCL: now also U3.38 (GPIO41/MTDI)
- net SDA: now also U3.39 (GPIO42/MTMS)
- net VDD3: now also J2.1 (Pin_1), TP3.1
- net GRN: now reaches U3.10 (GPIO17/ADC2_CH6)
- net GRN: now also J2.9 (Pin_9)
- net RED: now reaches U3.11 (GPIO18/ADC2_CH7)
- net RED: now also J2.10 (Pin_10)
- net BLU: now reaches U3.12 (GPIO8/ADC1_CH7)
- net BLU: now also J2.11 (Pin_11)
- net BTN_BALL: now reaches U3.4 (GPIO4/ADC1_CH3)
- net BTN_BALL: now also J2.3 (Pin_3)
- net RHT: now reaches U3.5 (GPIO5/ADC1_CH4)
- net RHT: now also J2.4 (Pin_4)
- net LFT: now reaches U3.6 (GPIO6/ADC1_CH5)
- net LFT: now also J2.5 (Pin_5)
- net DWN: now reaches U3.7 (GPIO7/ADC1_CH6)
- net DWN: now also J2.6 (Pin_6)
- net UP: now reaches U3.8 (GPIO15/ADC2_CH4/32K_P)
- net UP: now also J2.7 (Pin_7)
- net WHT: now reaches U3.9 (GPIO16/ADC2_CH5/32K_N)
- net WHT: now also J2.8 (Pin_8)

Commit message: ee
Parts:
- added SW35, SW66: SW_Push, Button_Switch_THT:SW_PUSH_6mm, symbol Switch:SW_Push
- TP3V1: renamed from TP3; footprint TestPoint:TestPoint_Pad_4.0x4.0mm -> TestPoint:TestPoint_Pad_2.5x2.5mm
- TP5V1: renamed from TP2; footprint TestPoint:TestPoint_Pad_4.0x4.0mm -> TestPoint:TestPoint_Pad_2.5x2.5mm
- TPGND1: renamed from TP1; footprint TestPoint:TestPoint_Pad_4.0x4.0mm -> TestPoint:TestPoint_Pad_2.5x2.5mm
Connections:
- net GND: now also SW35.2, SW66.1
- net at U3.3 (CHIP_PU): now also SW66.2
- net at U3.31 (GPIO0): now also SW35.1
