File: Mae_Keyboard_Dev_Kit/Atreus62.kicad_sch (KiCad schematic)
At the start: 144 parts, among them J1 gc9a01_DISPLAY, J2 Conn_01x11_Pin, SW1 SWITCH_PUSH, SW10 SWITCH_PUSH, SW11 SWITCH_PUSH, SW12 SWITCH_PUSH, SW13 SWITCH_PUSH, SW14 SWITCH_PUSH, SW15 SWITCH_PUSH, SW16 SWITCH_PUSH, SW17 SWITCH_PUSH, SW18 SWITCH_PUSH, SW19 SWITCH_PUSH, SW2 SWITCH_PUSH, SW20 SWITCH_PUSH, SW21 SWITCH_PUSH, SW22 SWITCH_PUSH, SW23 SWITCH_PUSH, SW24 SWITCH_PUSH, SW25 SWITCH_PUSH, SW26 SWITCH_PUSH, SW27 SWITCH_PUSH, SW28 SWITCH_PUSH, SW29 SWITCH_PUSH, SW3 SWITCH_PUSH, SW30 SWITCH_PUSH, SW31 SWITCH_PUSH, SW32 SWITCH_PUSH, SW33 SWITCH_PUSH, SW34 SWITCH_PUSH, SW35 SW_Push, SW36 SWITCH_PUSH, SW37 SWITCH_PUSH, SW38 SWITCH_PUSH, SW39 SWITCH_PUSH, SW4 SWITCH_PUSH, SW40 SWITCH_PUSH, SW41 SWITCH_PUSH, SW42 SWITCH_PUSH, SW43 SWITCH_PUSH, SW44 SWITCH_PUSH, SW45 SWITCH_PUSH, SW46 SWITCH_PUSH, SW47 SWITCH_PUSH, SW48 SWITCH_PUSH, SW49 SWITCH_PUSH, SW5 SWITCH_PUSH, SW50 SWITCH_PUSH, SW51 SWITCH_PUSH, SW52 SWITCH_PUSH, SW53 SWITCH_PUSH, SW54 SWITCH_PUSH, SW55 SWITCH_PUSH, SW56 SWITCH_PUSH, SW57 SWITCH_PUSH, SW58 SWITCH_PUSH, SW59 SWITCH_PUSH, SW6 SWITCH_PUSH, SW60 SWITCH_PUSH, SW61 SWITCH_PUSH, SW62 SWITCH_PUSH, SW63 SWITCH_PUSH, SW64 SWITCH_PUSH, SW65 SWITCH_PUSH, SW66 SW_Push, SW7 SWITCH_PUSH, SW8 SWITCH_PUSH, SW9 SWITCH_PUSH, U3 ESP32-S3-DevKitC

Commit message: update-integration
Parts:
- removed J2: Conn_01x11_Pin, Connector_PinSocket_2.54mm:PinSocket_1x11_P2.54mm_Vertical, symbol Connector:Conn_01x11_Pin
- removed SW35, SW66: SW_Push, Button_Switch_THT:SW_PUSH_6mm, symbol Switch:SW_Push
- added C1, C2: C_0805, PCM_Capacitor_SMD_AKL:C_0805_2012Metric, symbol PCM_Capacitor_AKL:C_0805
- added C3, C4: 1u, Capacitor_SMD:C_0805_2012Metric, symbol Device:C_Small
- added J2: Conn_01x06, ext:TP4056-18650, symbol Connector_Generic:Conn_01x06
- added Q1, Q2: BSS83P, PCM_Package_TO_SOT_SMD_AKL:SOT-23, symbol PCM_Transistor_MOSFET_AKL:BSS83P
- added TP3V2, TP3V3: TestPoint, TestPoint:TestPoint_Pad_1.5x1.5mm, symbol Connector:TestPoint
- added U1: NRF24L01_Breakout, RF_Module:nRF24L01_Breakout, symbol RF:NRF24L01_Breakout
- added U4: TLV73333PDBV, Package_TO_SOT_SMD:SOT-23-5, symbol Regulator_Linear:TLV73333PDBV
- D1, D10, D11, D12, D13, D14, D15, D16, D17, D18, D19, D2, D20, D21, D22, D23, D24, D25, D26, D27, D28, D29, D3, D30, D31, D33, D34, D35, D36, D37, D38, D39, D4, D40, D41, D42, D43, D44, D45, D46, D47, D48, D49, D5, D50, D51, D52, D53, D54, D55, D56, D57, D58, D59, D6, D60, D61, D62, D63, D64, D65, D7, D8, D9: footprint Diode_SMD:D_SOD-123 -> MaeLid:D_SOD-123
Connections:
- net BLU is gone; now on net COL3: U3.12 (GPIO8/ADC1_CH7)
- net DWN is gone; now on net DC: U3.7 (GPIO7/ADC1_CH6)
- net GRN is gone; now on net COL5: U3.10 (GPIO17/ADC2_CH6)
- net RED is gone; now on net COL4: U3.11 (GPIO18/ADC2_CH7)
- net UP is gone; now on net CS: U3.8 (GPIO15/ADC2_CH4/32K_P)
- net WHT is gone; now on net COL6: U3.9 (GPIO16/ADC2_CH5/32K_N)
- net +5V: now also J2.1 (Pin_1)
- net COL0: now also U3.15 (GPIO9/ADC1_CH8); no longer U3.27 (GPIO21)
- net COL1: now also U3.14 (GPIO46); no longer U3.28 (GPIO47)
- net COL10: now also U3.40 (GPIO2/ADC1_CH1); no longer U3.18 (GPIO12/ADC2_CH1)
- net COL11: now also U3.39 (GPIO42/MTMS); no longer U3.19 (GPIO13/ADC2_CH2)
- net COL12: now also U3.38 (GPIO41/MTDI); no longer U3.20 (GPIO14/ADC2_CH3)
- net COL2: now also U3.13 (GPIO3/ADC1_CH2); no longer U3.29 (GPIO48)
- net COL3: no longer U3.30 (GPIO45)
- net COL4: no longer U3.32 (GPIO35)
- net COL5: no longer U3.35 (GPIO38)
- net COL6: no longer U3.14 (GPIO46)
- net COL7: now also U3.43 (GPIO43/U0TXD); no longer U3.15 (GPIO9/ADC1_CH8)
- net COL8: now also U3.42 (GPIO44/U0RXD); no longer U3.16 (GPIO10/ADC1_CH9)
- net COL9: now also U3.41 (GPIO1/ADC1_CH0); no longer U3.17 (GPIO11/ADC2_CH0)
- net CS: no longer U3.41 (GPIO1/ADC1_CH0)
- net DC: no longer U3.40 (GPIO2/ADC1_CH1)
- net GND: now also C1.2, C2.2, C3.2, C4.2, J2.2 (Pin_2), J2.4 (Pin_4), U1.1 (GND), U4.2 (GND)
- net ROW0: now also U3.20 (GPIO14/ADC2_CH3); no longer U3.34 (GPIO37)
- net ROW1: now also U3.19 (GPIO13/ADC2_CH2); no longer U3.37 (GPIO40/MTDO)
- net ROW2: now also U3.18 (GPIO12/ADC2_CH1); no longer U3.36 (GPIO39/MTCK)
- net ROW3: now also U3.17 (GPIO11/ADC2_CH0); no longer U3.33 (GPIO36)
- net ROW4: now also U3.16 (GPIO10/ADC1_CH9); no longer U3.13 (GPIO3/ADC1_CH2)
- net RST: now also U3.35 (GPIO38); no longer U3.42 (GPIO44/U0RXD)
- net BTN_BALL renamed MISO
- net MISO: now also U1.7 (MISO)
- net LFT renamed SCK
- net SCK: now also J1.3 (Pin_3), U1.5 (SCK)
- net RHT renamed MOSI
- net MOSI: now also J1.4 (Pin_4), U1.6 (MOSI)
- removed net SCL: J1.3 (Pin_3), U3.38 (GPIO41/MTDI)
- removed net SDA: J1.4 (Pin_4), U3.39 (GPIO42/MTMS)
- net VDD3 renamed +3V3
- net +3V3: now also C4.1, Q1.2 (S), Q2.2 (S), U4.5 (OUT); no longer J1.1 (Pin_1)
- new net: TP3V2.1, U3.37 (GPIO40/MTDO)
- new net: TP3V3.1, U3.36 (GPIO39/MTCK)
- new net 33DISP: C2.1, J1.1 (Pin_1), Q2.3 (D)
- new net 33NRF: C1.1, Q1.3 (D), U1.2 (VCC)
- new net ALIM_DISP: Q2.1 (G), U3.32 (GPIO35)
- new net ALIM_NRF: Q1.1 (G), U3.33 (GPIO36)
- new net B+: J2.5 (Pin_5)
- new net B-: J2.6 (Pin_6)
- new net CE_NRF: U1.3 (CE), U3.28 (GPIO47)
- new net CS_NRF: U1.4 (~{CSN}), U3.29 (GPIO48)
- new net IRQ_NRF: U1.8 (IRQ), U3.30 (GPIO45)
- new net OUT+: C3.1, J2.3 (Pin_3), U4.1 (IN), U4.3 (EN)
Other:
- note removed: "Battery Level"
- note removed: "Quartz"
- moved on the sheet: J1, TP3V1, TP5V1, TPGND1, U3
