File: Mae_Keyboard_Dev_Kit/Atreus62.kicad_pcb (KiCad board)
At the start: 2 copper layers, 296.8 x 144.9 mm, 139 parts, among them J1 gc9a01_DISPLAY, J2 Conn_01x11_Pin, SW1 SWITCH_PUSH, SW10 SWITCH_PUSH, SW11 SWITCH_PUSH, SW12 SWITCH_PUSH, SW13 SWITCH_PUSH, SW14 SWITCH_PUSH, SW15 SWITCH_PUSH, SW16 SWITCH_PUSH, SW17 SWITCH_PUSH, SW18 SWITCH_PUSH, SW19 SWITCH_PUSH, SW2 SWITCH_PUSH, SW20 SWITCH_PUSH, SW21 SWITCH_PUSH, SW22 SWITCH_PUSH, SW23 SWITCH_PUSH, SW24 SWITCH_PUSH, SW25 SWITCH_PUSH, SW26 SWITCH_PUSH, SW27 SWITCH_PUSH, SW28 SWITCH_PUSH, SW29 SWITCH_PUSH, SW3 SWITCH_PUSH, SW30 SWITCH_PUSH, SW31 SWITCH_PUSH, SW32 SWITCH_PUSH, SW33 SWITCH_PUSH, SW34 SWITCH_PUSH, SW36 SWITCH_PUSH, SW37 SWITCH_PUSH, SW38 SWITCH_PUSH, SW39 SWITCH_PUSH, SW4 SWITCH_PUSH, SW40 SWITCH_PUSH, SW41 SWITCH_PUSH, SW42 SWITCH_PUSH, SW43 SWITCH_PUSH, SW44 SWITCH_PUSH, SW45 SWITCH_PUSH, SW46 SWITCH_PUSH, SW47 SWITCH_PUSH, SW48 SWITCH_PUSH, SW49 SWITCH_PUSH, SW5 SWITCH_PUSH, SW50 SWITCH_PUSH, SW51 SWITCH_PUSH, SW52 SWITCH_PUSH, SW53 SWITCH_PUSH, SW54 SWITCH_PUSH, SW55 SWITCH_PUSH, SW56 SWITCH_PUSH, SW57 SWITCH_PUSH, SW58 SWITCH_PUSH, SW59 SWITCH_PUSH, SW6 SWITCH_PUSH, SW60 SWITCH_PUSH, SW61 SWITCH_PUSH, SW62 SWITCH_PUSH, SW63 SWITCH_PUSH, SW64 SWITCH_PUSH, SW65 SWITCH_PUSH, SW7 SWITCH_PUSH, SW8 SWITCH_PUSH, SW9 SWITCH_PUSH, U3 ESP32-S3-DevKitC

Commit message: update
Parts:
- added TP3V: TestPoint, TestPoint:TestPoint_Pad_4.0x4.0mm, B.Cu at (148.7, 113.8)
- added TP5V: TestPoint, TestPoint:TestPoint_Pad_4.0x4.0mm, B.Cu at (168.8, 55.6)
- added TPGND: TestPoint, TestPoint:TestPoint_Pad_4.0x4.0mm, B.Cu at (174.2, 55.6)
- moved J2 25.4 mm to (135.6, 131.3), turned to 90 degrees
Connections:
- J2 pad 1: unconnected-(J2-Pin_1-Pad1) -> VDD3
- J2 pad 10: unconnected-(J2-Pin_10-Pad10) -> RED
- J2 pad 11: unconnected-(J2-Pin_11-Pad11) -> BLU
- J2 pad 2: unconnected-(J2-Pin_2-Pad2) -> GND
- J2 pad 3: unconnected-(J2-Pin_3-Pad3) -> BTN_BALL
- J2 pad 4: unconnected-(J2-Pin_4-Pad4) -> RHT
- J2 pad 5: unconnected-(J2-Pin_5-Pad5) -> LFT
- J2 pad 6: unconnected-(J2-Pin_6-Pad6) -> DWN
- J2 pad 7: unconnected-(J2-Pin_7-Pad7) -> UP
- J2 pad 8: unconnected-(J2-Pin_8-Pad8) -> WHT
- J2 pad 9: unconnected-(J2-Pin_9-Pad9) -> GRN
- U3 pad 10: unconnected-(U3-GPIO17/ADC2_CH6-Pad10) -> GRN
- U3 pad 11: unconnected-(U3-GPIO18/ADC2_CH7-Pad11) -> RED
- U3 pad 12: unconnected-(U3-GPIO8/ADC1_CH7-Pad12) -> BLU
- U3 pad 38: unconnected-(U3-GPIO41/MTDI-Pad38) -> SCL
- U3 pad 39: unconnected-(U3-GPIO42/MTMS-Pad39) -> SDA
- U3 pad 4: unconnected-(U3-GPIO4/ADC1_CH3-Pad4) -> BTN_BALL
- U3 pad 40: unconnected-(U3-GPIO2/ADC1_CH1-Pad40) -> DC
- U3 pad 41: unconnected-(U3-GPIO1/ADC1_CH0-Pad41) -> CS
- U3 pad 42: unconnected-(U3-GPIO44/U0RXD-Pad42) -> RST
- U3 pad 5: unconnected-(U3-GPIO5/ADC1_CH4-Pad5) -> RHT
- U3 pad 6: unconnected-(U3-GPIO6/ADC1_CH5-Pad6) -> LFT
- U3 pad 7: unconnected-(U3-GPIO7/ADC1_CH6-Pad7) -> DWN
- U3 pad 8: unconnected-(U3-GPIO15/ADC2_CH4/32K_P-Pad8) -> UP
- U3 pad 9: unconnected-(U3-GPIO16/ADC2_CH5/32K_N-Pad9) -> WHT
Routing:
- net BLU: track 0.00 -> 60.6 mm
- net RED: track 0.00 -> 56.7 mm
- net GRN: track 0.00 -> 54.5 mm
- net WHT: track 0.00 -> 52.4 mm
- net UP: track 0.00 -> 50.7 mm
- net DWN: track 0.00 -> 47.6 mm
- net LFT: track 0.00 -> 45.8 mm
- net VDD3: track 6.47 -> 50.9 mm, vias 0 -> 4
- net RHT: track 0.00 -> 43.9 mm
- net BTN_BALL: track 0.00 -> 42.3 mm
- net SCL: track 0.00 -> 19.4 mm
- net SDA: track 0.00 -> 15.8 mm
- net DC: track 0.00 -> 12.2 mm
- net +5V: track 0.00 -> 9.27 mm
- net CS: track 0.00 -> 8.80 mm
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
Commit message: ee
Parts:
- removed TP3V, TP5V, TPGND: TestPoint, TestPoint:TestPoint_Pad_4.0x4.0mm
- added REF**: LOGO, MaeLid:LOGO, F.Cu at (148.3, 136.1)
- added SW35: SW_Push, Button_Switch_THT:SW_PUSH_6mm, F.Cu at (125.5, 135.4)
- added SW66: SW_Push, Button_Switch_THT:SW_PUSH_6mm, F.Cu at (164.8, 135.4)
- added TP3V1: TestPoint, TestPoint:TestPoint_Pad_2.5x2.5mm, B.Cu at (148.8, 113.8)
- added TP5V1: TestPoint, TestPoint:TestPoint_Pad_2.5x2.5mm, B.Cu at (168.1, 55.7)
- added TPGND1: TestPoint, TestPoint:TestPoint_Pad_2.5x2.5mm, B.Cu at (174.2, 55.6)
- moved HS9 124.5 mm to (287.8, 134.4)
Connections:
- U3 pad 3: unconnected-(U3-CHIP_PU-Pad3) -> Net-(U3-CHIP_PU)
- U3 pad 31: unconnected-(U3-GPIO0-Pad31) -> Net-(U3-GPIO0)
Routing:
- net Net-(U3-CHIP_PU): track 0.00 -> 92.5 mm, vias 0 -> 2
- net Net-(U3-GPIO0): track 0.00 -> 87.6 mm, vias 0 -> 2
- net ROW1: track 489.9 -> 489.0 mm
- net GND: vias 2387 -> 2329
Other:
- board text added: "V. 1.1.0A"
- board text removed: "V. 1.0.0"

Commit message: send JLC
Routing:
- net COL6: track 208.7 -> 209.7 mm
