File: Mae_Keyboard_Dev_Kit/Atreus62.kicad_pcb (KiCad board)
At the start: 2 copper layers, 296.8 x 144.9 mm, 145 parts, among them J1 gc9a01_DISPLAY, J2 Conn_01x11_Pin, SW1 SWITCH_PUSH, SW10 SWITCH_PUSH, SW11 SWITCH_PUSH, SW12 SWITCH_PUSH, SW13 SWITCH_PUSH, SW14 SWITCH_PUSH, SW15 SWITCH_PUSH, SW16 SWITCH_PUSH, SW17 SWITCH_PUSH, SW18 SWITCH_PUSH, SW19 SWITCH_PUSH, SW2 SWITCH_PUSH, SW20 SWITCH_PUSH, SW21 SWITCH_PUSH, SW22 SWITCH_PUSH, SW23 SWITCH_PUSH, SW24 SWITCH_PUSH, SW25 SWITCH_PUSH, SW26 SWITCH_PUSH, SW27 SWITCH_PUSH, SW28 SWITCH_PUSH, SW29 SWITCH_PUSH, SW3 SWITCH_PUSH, SW30 SWITCH_PUSH, SW31 SWITCH_PUSH, SW32 SWITCH_PUSH, SW33 SWITCH_PUSH, SW34 SWITCH_PUSH, SW35 SW_Push, SW36 SWITCH_PUSH, SW37 SWITCH_PUSH, SW38 SWITCH_PUSH, SW39 SWITCH_PUSH, SW4 SWITCH_PUSH, SW40 SWITCH_PUSH, SW41 SWITCH_PUSH, SW42 SWITCH_PUSH, SW43 SWITCH_PUSH, SW44 SWITCH_PUSH, SW45 SWITCH_PUSH, SW46 SWITCH_PUSH, SW47 SWITCH_PUSH, SW48 SWITCH_PUSH, SW49 SWITCH_PUSH, SW5 SWITCH_PUSH, SW50 SWITCH_PUSH, SW51 SWITCH_PUSH, SW52 SWITCH_PUSH, SW53 SWITCH_PUSH, SW54 SWITCH_PUSH, SW55 SWITCH_PUSH, SW56 SWITCH_PUSH, SW57 SWITCH_PUSH, SW58 SWITCH_PUSH, SW59 SWITCH_PUSH, SW6 SWITCH_PUSH, SW60 SWITCH_PUSH, SW61 SWITCH_PUSH, SW62 SWITCH_PUSH, SW63 SWITCH_PUSH, SW64 SWITCH_PUSH, SW65 SWITCH_PUSH, SW66 SW_Push, SW7 SWITCH_PUSH, SW8 SWITCH_PUSH, SW9 SWITCH_PUSH, U3 ESP32-S3-DevKitC

Commit message: update-integration
Parts:
- removed REF**: LOGO, MaeLid:LOGO
- removed SW35, SW66: SW_Push, Button_Switch_THT:SW_PUSH_6mm
- added C1: C_0805, PCM_Capacitor_SMD_AKL:C_0805_2012Metric, B.Cu at (202.7, 141.6)
- added C2: C_0805, PCM_Capacitor_SMD_AKL:C_0805_2012Metric, B.Cu at (219.0, 158.7)
- added C3: 1u, Capacitor_SMD:C_0805_2012Metric, B.Cu at (286.4, 214.1)
- added C4: 1u, Capacitor_SMD:C_0805_2012Metric, B.Cu at (284.0, 210.0)
- added Q1: BSS83P, PCM_Package_TO_SOT_SMD_AKL:SOT-23, B.Cu at (98.1, 230.1)
- added Q2: BSS83P, PCM_Package_TO_SOT_SMD_AKL:SOT-23, B.Cu at (93.6, 230.1)
- added TP3V2: TestPoint, TestPoint:TestPoint_Pad_1.5x1.5mm, F.Cu at (269.7, 236.7)
- added TP3V3: TestPoint, TestPoint:TestPoint_Pad_1.5x1.5mm, F.Cu at (264.5, 236.7)
- added U1: NRF24L01_Breakout, RF_Module:nRF24L01_Breakout, F.Cu at (206.9, 143.1)
- added U4: TLV73333PDBV, Package_TO_SOT_SMD:SOT-23-5, B.Cu at (283.0, 214.0)
- D1, D10, D11, D12, D13, D14, D15, D16, D17, D18, D19, D2, D20, D21, D22, D23, D24, D25, D26, D27, D28, D29, D3, D30, D31, D33, D34, D35, D36, D37, D38, D39, D4, D40, D41, D42, D43, D44, D45, D46, D47, D48, D49, D5, D50, D51, D52, D53, D54, D55, D56, D57, D58, D59, D6, D60, D61, D62, D63, D64, D65, D7, D8, D9: footprint Diode_SMD:D_SOD-123 -> MaeLid:D_SOD-123
- J2: value Conn_01x11_Pin -> Conn_01x06; footprint Connector_PinSocket_2.54mm:PinSocket_1x11_P2.54mm_Vertical -> ext:TP4056-18650
- moved TPGND1 183.8 mm to (68.2, 205.7), turned to 0 degrees
- moved TP5V1 176.8 mm to (74.3, 205.6), turned to 0 degrees
- moved TP3V1 162.7 mm to (280.1, 209.9)
- moved J2 150.4 mm to (259.3, 217.0), turned to 0 degrees
- moved U3 109.5 mm to (126.8, 211.4), turned to -90 degrees
- moved D50 91.2 mm to (321.3, 155.8)
- moved D29 90.4 mm to (184.1, 185.3)
- moved D54 90.3 mm to (330.8, 135.3)
- moved D6 89.7 mm to (108.4, 106.0)
- moved D1 89.1 mm to (72.0, 115.8)
- moved D21 89.0 mm to (179.8, 112.9), turned to -10 degrees
- moved D65 88.7 mm to (208.7, 171.9)
- moved D27 88.7 mm to (193.1, 139.0)
- moved D53 88.4 mm to (339.5, 114.8)
- moved D26 88.3 mm to (196.7, 119.5)
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Connections:
- J1 pad 1: VDD3 -> 33DISP
- J1 pad 3: SCL -> SCK
- J1 pad 4: SDA -> MOSI
- J2 pad 1: VDD3 -> +5V
- J2 pad 3: BTN_BALL -> OUT+
- J2 pad 4: RHT -> GND
- J2 pad 5: LFT -> B+
- J2 pad 6: DWN -> B-
- TP3V1 pad 1: VDD3 -> +3V3
- U3 pad 1: VDD3 -> +3V3
- U3 pad 10: GRN -> COL5
- U3 pad 11: RED -> COL4
- U3 pad 12: BLU -> COL3
- U3 pad 13: ROW4 -> COL2
- U3 pad 14: COL6 -> COL1
- U3 pad 15: COL7 -> COL0
- U3 pad 16: COL8 -> ROW4
- U3 pad 17: COL9 -> ROW3
- U3 pad 18: COL10 -> ROW2
- U3 pad 19: COL11 -> ROW1
- U3 pad 2: VDD3 -> +3V3
- U3 pad 20: COL12 -> ROW0
- U3 pad 27: COL0 -> unconnected-(U3-GPIO21-Pad27)
- U3 pad 28: COL1 -> CE_NRF
- U3 pad 29: COL2 -> CS_NRF
- U3 pad 3: Net-(U3-CHIP_PU) -> unconnected-(U3-CHIP_PU-Pad3)
- U3 pad 30: COL3 -> IRQ_NRF
- U3 pad 31: Net-(U3-GPIO0) -> unconnected-(U3-GPIO0-Pad31)
- U3 pad 32: COL4 -> ALIM_DISP
- U3 pad 33: ROW3 -> ALIM_NRF
- U3 pad 34: ROW0 -> unconnected-(U3-GPIO37-Pad34)
- U3 pad 35: COL5 -> RST
- U3 pad 36: ROW2 -> Net-(U3-GPIO39/MTCK)
- U3 pad 37: ROW1 -> Net-(U3-GPIO40/MTDO)
- U3 pad 38: SCL -> COL12
- U3 pad 39: SDA -> COL11
- U3 pad 4: BTN_BALL -> MISO
- U3 pad 40: DC -> COL10
- U3 pad 41: CS -> COL9
- U3 pad 42: RST -> COL8
- U3 pad 43: unconnected-(U3-GPIO43/U0TXD-Pad43) -> COL7
- U3 pad 5: RHT -> MOSI
- U3 pad 6: LFT -> SCK
- U3 pad 7: DWN -> DC
- U3 pad 8: UP -> CS
- U3 pad 9: WHT -> COL6
Routing:
- net ROW4: track 1039.7 -> 0.00 mm, vias 6 -> 0
- net ROW3: track 572.8 -> 0.00 mm, vias 19 -> 0
- net ROW0: track 561.7 -> 0.00 mm
- net ROW1: track 489.4 -> 0.00 mm, vias 24 -> 0
- net ROW2: track 396.7 -> 0.00 mm, vias 22 -> 0
- net COL12: track 240.2 -> 0.00 mm
- net COL11: track 220.0 -> 0.00 mm
- net COL0: track 213.0 -> 0.00 mm, vias 2 -> 0
- net COL6: track 209.7 -> 0.00 mm, vias 2 -> 0
- net COL10: track 201.4 -> 0.00 mm, vias 6 -> 0
- net COL1: track 187.7 -> 0.00 mm, vias 2 -> 0
- net COL2: track 177.4 -> 0.00 mm, vias 2 -> 0
- net COL9: track 169.0 -> 0.00 mm, vias 4 -> 0
- net COL3: track 161.4 -> 0.00 mm
- net COL8: track 146.0 -> 0.00 mm, vias 2 -> 0
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Other:
- board size 296.8 x 144.9 mm -> 296.8 x 145 mm
- board text added: "KaSe"
