File: V2/KaSe/KaSe.kicad_pcb (KiCad board)
At the start: 2 copper layers, 296.8 x 145 mm, 158 parts, among them J1 gc9a01_DISPLAY, J2 Conn_01x06, J4 Conn_01x03, J5 Conn_01x03, Q1 BSS83P, Q2 BSS83P, SW1 SWITCH_PUSH, SW10 SWITCH_PUSH, SW11 SWITCH_PUSH, SW12 SWITCH_PUSH, SW13 SWITCH_PUSH, SW14 SWITCH_PUSH, SW15 SWITCH_PUSH, SW16 SWITCH_PUSH, SW17 SWITCH_PUSH, SW18 SWITCH_PUSH, SW19 SWITCH_PUSH, SW2 SWITCH_PUSH, SW20 SWITCH_PUSH, SW21 SWITCH_PUSH, SW22 SWITCH_PUSH, SW23 SWITCH_PUSH, SW24 SWITCH_PUSH, SW25 SWITCH_PUSH, SW26 SWITCH_PUSH, SW27 SWITCH_PUSH, SW28 SWITCH_PUSH, SW29 SWITCH_PUSH, SW3 SWITCH_PUSH, SW30 SWITCH_PUSH, SW31 SWITCH_PUSH, SW32 SWITCH_PUSH, SW33 SWITCH_PUSH, SW34 SWITCH_PUSH, SW36 SWITCH_PUSH, SW37 SWITCH_PUSH, SW38 SWITCH_PUSH, SW39 SWITCH_PUSH, SW4 SWITCH_PUSH, SW40 SWITCH_PUSH, SW41 SWITCH_PUSH, SW42 SWITCH_PUSH, SW43 SWITCH_PUSH, SW44 SWITCH_PUSH, SW45 SWITCH_PUSH, SW46 SWITCH_PUSH, SW47 SWITCH_PUSH, SW48 SWITCH_PUSH, SW49 SWITCH_PUSH, SW5 SWITCH_PUSH, SW50 SWITCH_PUSH, SW51 SWITCH_PUSH, SW52 SWITCH_PUSH, SW53 SWITCH_PUSH, SW54 SWITCH_PUSH, SW55 SWITCH_PUSH, SW56 SWITCH_PUSH, SW57 SWITCH_PUSH, SW58 SWITCH_PUSH, SW59 SWITCH_PUSH, SW6 SWITCH_PUSH, SW60 SWITCH_PUSH, SW61 SWITCH_PUSH, SW62 SWITCH_PUSH, SW63 SWITCH_PUSH, SW64 SWITCH_PUSH, SW65 SWITCH_PUSH, SW7 SWITCH_PUSH, SW8 SWITCH_PUSH, SW9 SWITCH_PUSH, U1 NRF24L01_Breakout, U2 AP130-33SA, U3 ESP32-S3-DevKitC, U4 TLV73333PDBV

Commit message: add i2c display ssd1306 and clean up for print
Parts:
- added J3: Conn_01x04_Pin, Connector_PinHeader_2.54mm:PinHeader_1x04_P2.54mm_Vertical, F.Cu at (216.3, 158.4)
- moved C2 2.12 mm to (221.1, 159.0), turned to 0 degrees
Routing:
- net ROW0: track 0.00 -> 593.6 mm, vias 0 -> 4
- net ROW4: track 0.00 -> 515.7 mm, vias 0 -> 9
- net ROW3: track 0.00 -> 505.1 mm, vias 0 -> 14
- net ROW2: track 0.00 -> 448.3 mm, vias 0 -> 9
- net ROW1: track 0.00 -> 431.7 mm, vias 0 -> 9
- net COL12: track 0.00 -> 408.3 mm, vias 0 -> 4
- net COL11: track 0.00 -> 368.5 mm, vias 0 -> 3
- net COL10: track 0.00 -> 346.9 mm, vias 0 -> 2
- net COL9: track 0.00 -> 286.3 mm, vias 0 -> 6
- net COL8: track 0.00 -> 258.8 mm, vias 0 -> 4
- net COL6: track 0.00 -> 257.4 mm
- net +5V: track 0.00 -> 236.3 mm
- net COL7: track 0.00 -> 234.5 mm, vias 0 -> 4
- net IRQ_NRF: track 0.00 -> 231.9 mm, vias 0 -> 2
- net +3V3: track 0.00 -> 227.1 mm, vias 0 -> 2
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
Commit message: u
Routing:
- net ROW0: track 593.6 -> 562.1 mm
- net ROW1: track 431.7 -> 428.1 mm
Other:
- board text added: "C0"
- board text added: "C1"
- board text added: "C2"
- board text added: "C3"
- board text added: "C4"
- board text added: "C5"
- board text added: "C6"
- board text added: "CS"
- board text added: "DC"
- board text added: "MISO"
- board text added: "MOSI"
- board text added: "R0"
- board text added: "R1"
- board text added: "R2"
- board text added: "R3"
- board text added: "R4"
- board text added: "SCK"
